File: extras/SI4844_LCD16x02.sch (EAGLE design)
At the start: 9 parts, among them M1 ARDUINO-NANO-3.0

Commit message: SI4844 Arduino Library
Parts:
- removed U$1: SI4844SI4844, SI4844_PU2CLR:SI4844SI4844
- added B1: SPARKFUN_LOGIC_LEVEL_CONVERTERLOCK, SparkFun-Boards:SPARKFUN_LOGIC_LEVEL_CONVERTERLOCK
- added C1, C2: 22pF, capacitor-wima:C2,5-3
- added C3, C6: 100nF, capacitor-wima:C2,5-3
- added C4, C5: 4.7uF, capacitor-wima:C2,5-3
- added C7: 470nF, capacitor-wima:C2,5-3
- added FM: (no value), discrete:ANTENNA
- added J1: (no value), SparkFun-Connectors:AUDIO_JACK_2.5MMSPECIAL_POGO_PINS
- added L1: L, adafruit:L
- added L2: (no value), ngspice-simulation:L
- added Q1: (no value), special:XTAL
- added R1, R2: 3.3K, Resistor:R-US_AXIAL-7.2MM-PITCH
- added R3: 100k, SparkFun-Resistors:POTENTIOMETER-PTH-9MM-1/20W-20%
- SI1: value SI4844SI4844 -> SI4844; device SI4844_PU2CLR:SI4844SI4844 -> SI4844_PU2CLR:SI4844
Connections:
- new net N$12: C1.2, Q1.1, SI1.XTALI
- new net N$13: C2.2, Q1.2, SI1.XTALO
- new net N$14: FM.1, L1.2, SI1.FMI
- new net N$15: C7.1, SI1.AMI
- new net N$16: C7.2, L1.1, L2.2
- new net N$17: C5.1, J1.RIGHT
- new net N$18: C4.1, J1.LEFT
- new net N$19: B1.LV_TXI_2, R2.1, SI1.SCLK
- new net N$20: C3.2, SI1.DBYP
- new net N$21: B1.LV_RXO_2, R1.1, SI1.SDIO
- new net N$22: B1.LV_RXO_1, C6.1, SI1.RST
- new net N$23: B1.HV_TXO_2, M1.A5
- new net N$24: B1.HV_RXI_2, M1.A4
- new net N$25: B1.LV_TXI_1, SI1.IRQ
- new net N$26: B1.HV_TXO_1, M1.D2
- new net N$27: B1.HV_RXI_1, M1.D12/MISO
- new net N$28: R3.E, SI1.TUNE1
- new net N$29: R3.S, SI1.TUNE2
- new net N$30: SI1.BAND
- new net N$31: C4.2, SI1.LOUT
- new net N$32: C5.2, SI1.ROUT
- net GND: now also B1.GND, B1.GND@2, C1.1, C2.1, C6.2, J1.SLEEVE, L2.1, R3.A, SI1.GND1, SI1.GND2, SI1.NC3, SI1.NC4, SI1.RFGND
- net N$11: now also M1.D3; no longer M1.D2
- net VCC: now also B1.HV, B1.LV, C3.1, R1.2, R2.2, SI1.VDD1, SI1.VDD2
Other:
- note added: "Bi-directional logic level converter"
- note added: "Ferrite Antenna"
- note added: "IRQ / Interrupt"
- note added: "L1 100mH"
- note added: "RST"
- note added: "SCLK"
- note added: "SDIO"
- moved on the sheet: BAND_DOWN, BAN_UP, LCD1, M1, VOL_DOWN, VOL_UP, VR1
