File: extras/schematic_eagle_basic.sch (EAGLE design)
At the start: 3 parts, among them M1 ARDUINO-PRO-MINI-3.3V, P1 SOP63P600X175-24N, P2 SOP63P600X175-24N

Commit message: SI4844 Arduino Library
Parts:
- removed P1, P2: SOP63P600X175-24N, SOP63P600X175-24N:SOP63P600X175-24N
- added BAND_DOWN, BAND_UP, VOL_DOWN, VOL_UP: (no value), adafruit:SWITCH_PUSHBUTTONC&K_KSS
- added J2_SDIO, J3_SCLK, J4_RST, J5_IRQ: (no value), SparkFun-Connectors:CONN_01
- added U$1: DISPLAY-OLED-128X64-I2C, diy-modules:DISPLAY-OLED-128X64-I2C
Connections:
- removed net SCL: M1.A5
- removed net SDA: M1.A4
- new net GND: BAND_DOWN.P$2, BAND_UP.P$2, M1.GND.2, U$1.GND, VOL_DOWN.P$1, VOL_UP.P$1
- new net N$1: J3_SCLK.1, M1.A5, U$1.SCL
- new net N$2: J4_RST.1, M1.D12
- new net N$3: J2_SDIO.1, M1.A4, U$1.SDA
- new net N$4: J5_IRQ.1, M1.D2
- new net N$5: M1.D11, VOL_UP.P$2
- new net N$7: BAND_DOWN.P$1, M1.D9
- new net N$8: BAND_UP.P$1, M1.D8
- new net N$9: M1.D10, VOL_DOWN.P$2
- new net VCC: M1.VCC, U$1.VCC
Other:
- note added: "SI4844"
- note removed: "to SI4844 pin 16"
- note removed: "to SI4844 pin 17"
- moved on the sheet: M1
