File: extras/KiCad/SI4844_STM32/SI4844_STM32.kicad_sch (KiCad schematic)
At the start: 17 parts, among them J1 AudioJack2_Ground, U1 STM32F103C8Tx, Y1 Crystal

Commit message: Doc
Parts:
- added R3: 100K, symbol Device:R
Connections:
- net at C7.1, SI1.RST: now also R3.1; no longer U1.25 (PB12)
- new net: R3.2, U1.25 (PB12)
Other:
- moved on the sheet: AE1
Changed lines of the file:
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@@
   (junction (at 147.32 93.98) (diameter 0) (color 0 0 0 0)
   )
+  (junction (at 115.57 119.38) (diameter 0) (color 0 0 0 0)
+  )
+  (junction (at 69.85 109.22) (diameter 0) (color 0 0 0 0)
+  )
+  (junction (at 162.56 113.03) (diameter 0) (color 0 0 0 0)
+  )
+  (junction (at 107.95 81.28) (diameter 0) (color 0 0 0 0)
+  )
+  (junction (at 125.73 93.98) (diameter 0) (color 0 0 0 0)
+  )
+  (junction (at 74.93 130.81) (diameter 0) (color 0 0 0 0)
+  )
+  (junction (at 69.85 114.3) (diameter 0) (color 0 0 0 0)
+  )
+  (junction (at 125.73 86.36) (diameter 0) (color 0 0 0 0)
+  )
+  (junction (at 140.97 125.73) (diameter 0) (color 0 0 0 0)
+  )
+  (junction (at 161.29 92.71) (diameter 0) (color 0 0 0 0)
+  )
   (junction (at 59.69 99.06) (diameter 0) (color 0 0 0 0)
   )
-  (junction (at 140.97 125.73) (diameter 0) (color 0 0 0 0)
-  )
-  (junction (at 115.57 119.38) (diameter 0) (color 0 0 0 0)
-  )
-  (junction (at 69.85 109.22) (diameter 0) (color 0 0 0 0)
-  )
-  (junction (at 162.56 113.03) (diameter 0) (color 0 0 0 0)
-  )
-  (junction (at 107.95 81.28) (diameter 0) (color 0 0 0 0)
-  )
-  (junction (at 125.73 93.98) (diameter 0) (color 0 0 0 0)
-  )
-  (junction (at 74.93 130.81) (diameter 0) (color 0 0 0 0)
-  )
-  (junction (at 69.85 114.3) (diameter 0) (color 0 0 0 0)
-  )
-  (junction (at 125.73 86.36) (diameter 0) (color 0 0 0 0)
-  )
-  (junction (at 161.29 92.71) (diameter 0) (color 0 0 0 0)
-  )
   (junction (at 132.08 73.66) (diameter 0) (color 0 0 0 0)
   )
@@
     (stroke (width 0) (type default))
   )
+  (wire (pts (xy 107.95 109.22) (xy 124.46 109.22))
+    (stroke (width 0) (type default))
+  )
   (wire (pts (xy 147.32 86.36) (xy 147.32 93.98))
     (stroke (width 0) (type default))
@@
     (stroke (width 0) (type default))
   )
-  (wire (pts (xy 107.95 109.22) (xy 124.46 109.22))
+  (wire (pts (xy 140.97 125.73) (xy 156.21 125.73))
     (stroke (width 0) (type default))
   )
@@
     (stroke (width 0) (type default))
   )
-  (wire (pts (xy 140.97 125.73) (xy 182.88 125.73))
-    (stroke (width 0) (type default))
-  )
   (wire (pts (xy 115.57 55.88) (xy 115.57 68.58))
     (stroke (width 0) (type default))
@@
     (stroke (width 0) (type default))
   )
+  (wire (pts (xy 107.95 88.9) (xy 120.65 88.9))
+    (stroke (width 0) (type default))
+  )
+  (wire (pts (xy 215.9 67.31) (xy 232.41 67.31))
+    (stroke (width 0) (type default))
+  )
+  (wire (pts (xy 22.86 97.79) (xy 22.86 99.06))
+    (stroke (width 0) (type default))
+  )
+  (wire (pts (xy 107.95 62.23) (xy 109.22 62.23))
+    (stroke (width 0) (type default))
+  )
+  (wire (pts (xy 45.72 78.74) (xy 77.47 78.74))
+    (stroke (width 0) (type default))
+  )
+  (wire (pts (xy 147.32 93.98) (xy 147.32 97.79))
+    (stroke (width 0) (type default))
+  )
+  (wire (pts (xy 74.93 129.54) (xy 74.93 130.81))
+    (stroke (width 0) (type default))
+  )
+  (wire (pts (xy 198.12 57.15) (xy 198.12 62.23))
+    (stroke (width 0) (type default))
+  )
+  (wire (pts (xy 107.95 99.06) (xy 134.62 99.06))
+    (stroke (width 0) (type default))
+  )
   (wire (pts (xy 22.86 99.06) (xy 59.69 99.06))
     (stroke (width 0) (type default))
   )
-  (wire (pts (xy 107.95 88.9) (xy 120.65 88.9))
-    (stroke (width 0) (type default))
-  )
-  (wire (pts (xy 215.9 67.31) (xy 232.41 67.31))
-    (stroke (width 0) (type default))
-  )
-  (wire (pts (xy 107.95 62.23) (xy 109.22 62.23))
-    (stroke (width 0) (type default))
-  )
-  (wire (pts (xy 45.72 78.74) (xy 77.47 78.74))
-    (stroke (width 0) (type default))
-  )
-  (wire (pts (xy 147.32 93.98) (xy 147.32 97.79))
-    (stroke (width 0) (type default))
-  )
-  (wire (pts (xy 74.93 129.54) (xy 74.93 130.81))
-    (stroke (width 0) (type default))
-  )
-  (wire (pts (xy 198.12 57.15) (xy 198.12 62.23))
-    (stroke (width 0) (type default))
-  )
-  (wire (pts (xy 107.95 99.06) (xy 134.62 99.06))
+  (wire (pts (xy 163.83 125.73) (xy 182.88 125.73))
     (stroke (width 0) (type default))
   )
@@
   )
   (wire (pts (xy 52.07 66.04) (xy 52.07 73.66))
-    (stroke (width 0) (type default))
-  )
-  (wire (pts (xy 22.86 100.33) (xy 22.86 99.06))
     (stroke (width 0) (type default))
   )
@@
         (path "/a0d8c9a3-7eb8-440c-942e-981585e19cdf"
           (reference "#PWR010") (unit 1)
+        )
+      )
+    )
+  )
+  (symbol (lib_id "Device:R") (at 160.02 125.73 90) (mirror x) (unit 1)
+    (in_bom yes) (on_board yes) (dnp no)
+    (property "Reference" "R3" (at 161.29 121.92 90)
+      (effects (font (size 1.27 1.27)) (justify left))
+    )
+    (property "Value" "100K" (at 162.56 128.27 90)
+      (effects (font (size 1.27 1.27)) (justify left))
+    )
+    (property "Footprint" "" (at 160.02 123.952 90)
+      (effects (font (size 1.27 1.27)) hide)
+    )
+    (property "Datasheet" "~" (at 160.02 125.73 0)
+      (effects (font (size 1.27 1.27)) hide)
+    )
+    (pin "1")
+    (pin "2")
+    (instances
+      (project "SI4844_STM32"
+        (path "/a0d8c9a3-7eb8-440c-942e-981585e19cdf"
+          (reference "R3") (unit 1)
         )
       )
@@
     )
   )
-  (symbol (lib_id "Device:Antenna") (at 22.86 95.25 0) (unit 1)
-    (in_bom yes) (on_board yes) (dnp no) (fields_autoplaced)
-    (property "Reference" "AE1" (at 25.4 94.615 0)
-      (effects (font (size 1.27 1.27)) (justify left))
-    )
-    (property "Value" "Antenna" (at 25.4 97.155 0)
-      (effects (font (size 1.27 1.27)) (justify left))
-    )
-    (property "Footprint" "" (at 22.86 95.25 0)
-      (effects (font (size 1.27 1.27)) hide)
-    )
-    (property "Datasheet" "~" (at 22.86 95.25 0)
-      (effects (font (size 1.27 1.27)) hide)
-    )
+  (symbol (lib_id "Device:Antenna") (at 22.86 92.71 0) (unit 1)
+    (in_bom yes) (on_board yes) (dnp no) (fields_autoplaced)
+    (property "Reference" "AE1" (at 25.4 92.075 0)
+      (effects (font (size 1.27 1.27)) (justify left))
+    )
+    (property "Value" "Antenna" (at 25.4 94.615 0)
+      (effects (font (size 1.27 1.27)) (justify left))
+    )
+    (property "Footprint" "" (at 22.86 92.71 0)
+      (effects (font (size 1.27 1.27)) hide)
+    )
+    (property "Datasheet" "~" (at 22.86 92.71 0)
+      (effects (font (size 1.27 1.27)) hide)
+    )
