File: extras/KiCad/SI4827_BASIC_SETUP/si4827.kicad_sch (KiCad schematic)
At the start: 19 parts, among them J1 MCU_INTERRUP, J2 MCU_RESET, J3 MCU_I2C_SDIO, J4 MCU_I2C_SCLK, J5 AudioJack2, U1 SI4827, Y1 32.768kHz

Commit message: Doc
Connections:
- net at VR1.P$2 (S): now also U1.3 (TUNE2); no longer U1.2 (TUNE1)
- net at VR1.P$3 (A): now also U1.2 (TUNE1); no longer U1.3 (TUNE2)
Other:
- moved on the sheet: VR1
Changed lines of the file:
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@@
+    (stroke (width 0) (type default))
+  )
+  (wire (pts (xy 55.88 35.56) (xy 68.58 35.56))
     (stroke (width 0) (type default))
   )
@@
     (stroke (width 0) (type default))
   )
-  (wire (pts (xy 59.69 21.59) (xy 59.69 19.05))
-    (stroke (width 0) (type default))
-  )
   (wire (pts (xy 68.58 45.72) (xy 43.18 45.72))
     (stroke (width 0) (type default))
@@
     (stroke (width 0) (type default))
   )
-  (wire (pts (xy 43.18 21.59) (xy 43.18 38.1))
-    (stroke (width 0) (type default))
-  )
   (wire (pts (xy 96.52 45.72) (xy 101.6 45.72))
     (stroke (width 0) (type default))
@@
     (stroke (width 0) (type default))
   )
+  (wire (pts (xy 68.58 38.1) (xy 48.26 38.1))
+    (stroke (width 0) (type default))
+  )
   (wire (pts (xy 142.24 39.37) (xy 142.24 43.18))
     (stroke (width 0) (type default))
@@
     (stroke (width 0) (type default))
   )
-  (wire (pts (xy 50.8 35.56) (xy 68.58 35.56))
-    (stroke (width 0) (type default))
-  )
   (wire (pts (xy 30.48 19.05) (xy 30.48 22.86))
     (stroke (width 0) (type default))
@@
     (stroke (width 0) (type default))
   )
+  (wire (pts (xy 48.26 38.1) (xy 48.26 26.67))
+    (stroke (width 0) (type default))
+  )
   (wire (pts (xy 109.22 69.85) (xy 111.76 69.85))
     (stroke (width 0) (type default))
@@
     (stroke (width 0) (type default))
   )
-  (wire (pts (xy 43.18 38.1) (xy 68.58 38.1))
-    (stroke (width 0) (type default))
-  )
-  (wire (pts (xy 58.42 21.59) (xy 59.69 21.59))
+  (wire (pts (xy 40.64 19.05) (xy 40.64 21.59))
     (stroke (width 0) (type default))
   )
@@
     (stroke (width 0) (type default))
   )
-  (wire (pts (xy 50.8 26.67) (xy 50.8 35.56))
+  (wire (pts (xy 55.88 21.59) (xy 55.88 35.56))
     (stroke (width 0) (type default))
   )
@@
   (symbol (lib_id "Connector:Conn_01x01_Pin") (at 60.96 33.02 0) (unit 1)
     (in_bom yes) (on_board yes) (dnp no)
-    (property "Reference" "J1" (at 61.595 27.94 0)
-      (effects (font (size 1.27 1.27)))
-    )
-    (property "Value" "MCU_INTERRUP" (at 60.96 30.48 0)
+    (property "Reference" "J1" (at 66.04 30.48 0)
+      (effects (font (size 1.27 1.27)))
+    )
+    (property "Value" "MCU_INTERRUP" (at 64.77 27.94 0)
       (effects (font (size 1 1)))
     )
@@
     )
   )
-  (symbol (lib_id "power:GND") (at 59.69 19.05 180) (unit 1)
-    (in_bom yes) (on_board yes) (dnp no) (fields_autoplaced)
-    (property "Reference" "#PWR03" (at 59.69 12.7 0)
-      (effects (font (size 1.27 1.27)) hide)
-    )
-    (property "Value" "GND" (at 59.69 13.97 0)
-      (effects (font (size 1.27 1.27)))
-    )
-    (property "Footprint" "" (at 59.69 19.05 0)
-      (effects (font (size 1.27 1.27)) hide)
-    )
-    (property "Datasheet" "" (at 59.69 19.05 0)
+  (symbol (lib_id "power:GND") (at 40.64 19.05 180) (unit 1)
+    (in_bom yes) (on_board yes) (dnp no) (fields_autoplaced)
+    (property "Reference" "#PWR03" (at 40.64 12.7 0)
+      (effects (font (size 1.27 1.27)) hide)
+    )
+    (property "Value" "GND" (at 40.64 13.97 0)
+      (effects (font (size 1.27 1.27)))
+    )
+    (property "Footprint" "" (at 40.64 19.05 0)
+      (effects (font (size 1.27 1.27)) hide)
+    )
+    (property "Datasheet" "" (at 40.64 19.05 0)
       (effects (font (size 1.27 1.27)) hide)
     )
@@
     )
   )
-  (symbol (lib_id "SI4844:POTENTIOMETER-PTH-9MM-1/20W-20%") (at 50.8 21.59 270) (unit 1)
-    (in_bom yes) (on_board yes) (dnp no) (fields_autoplaced)
-    (property "Reference" "VR1" (at 50.8 17.78 90)
+  (symbol (lib_id "SI4844:POTENTIOMETER-PTH-9MM-1/20W-20%") (at 48.26 21.59 90) (mirror x) (unit 1)
+    (in_bom yes) (on_board yes) (dnp no)
+    (property "Reference" "VR1" (at 48.26 17.78 90)
       (effects (font (size 1.778 1.778)))
     )
-    (property "Value" "~" (at 50.8 20.32 90)
+    (property "Value" "~" (at 48.26 20.32 90)
       (effects (font (size 1.778 1.778)) (justify bottom) hide)
     )
-    (property "Footprint" "SI4844_01:POT-PTH-ALPS" (at 50.8 21.59 0)
-      (effects (font (size 1.27 1.27)) hide)
-    )
-    (property "Datasheet" "" (at 50.8 21.59 0)
-      (effects (font (size 1.27 1.27)) hide)
-    )
+    (property "Footprint" "SI4844_01:POT-PTH-ALPS" (at 48.26 21.59 0)
+      (effects (font (size 1.27 1.27)) hide)
+    )
+    (property "Datasheet" "" (at 48.26 21.59 0)
+      (effects (font (size 1.27 1.27)) hide)
+    )
