File: extras/KiCad/mechanical_band_setup/mechanical_band_setup.kicad_sch (KiCad schematic)
At the start: 14 parts

Commit message: doc
Parts:
- R10, R3, R6, R7, R9: value 10K -> 20K
- R13: value 53K -> 63K
- R2: value 200K -> 160K
- R4: value 30K -> 10K
- R5: value 30K -> 40K
Other:
- note added: "227K"
- note added: "247K"
- note added: "257K"
- note added: "297K"
- note added: "317K"
- note added: "337K"
- note added: "377K"
- note added: "417K"
- note added: "437K"
- note added: "500K"
- note added: "Si48XX BAND"
- note added: "Si48XX TUNE1"
- note added: "| Band Name | Narrow Frequency Range | Wide Frequency Range | | ---------- | ------------------------| ---------------------- | | FM1 | 87-108 MHz | 64-108 MHZ | | FM5 | 64-87 MHz | 76-108 MHZ | | AM1 | 520-1710 KHZ | ------------ | | AM2 | 522-1620 KHZ | ------------ | | SW1 | 5.6-6.4 MHz | 3.2-7.6 MHz | | SW3 | 6.8-7.6 MHz | 3.2-100 MHz | | SW5 | 9.2.4-10.0 MHz | 5.9-18.0 MHz | | SW7 | 11.45-12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"
- note removed: "267"
- note removed: "277K"
- note removed: "307K"
- note removed: "347K"
- note removed: "367K"
- note removed: "387K"
- note removed: "407K"
- note removed: "427K"
- note removed: "447K"
- note removed: "Si4825 BAND(PIN 4)"
- note removed: "Si4825 TUNE1(PIN 2)"
- note removed: "| Band Name | Narrow Frequency Range | Wide Frequency Range | | ---------- | ------------------------| ---------------------- | | FM3 | 87-108 MHz (75 µs) | | | AM5 | 510-1750 kHz (10kHz) | | | SW1 | 2.30-2.49 MHz | 2.3-10.0 MHz | | SW4 | 4.75-5.06 MHz | 3.7-12.5 MHz | | SW8 | 7.1-7.6 MHz | 5.9-9.50 MHz | | SW9 | 9.2-10 MHz | 5.9-18.0 MHz | | SW10 | 11.45-12.25 MHz | 7.0-16.0 MHz | | SW12 | 13.4-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"
- title: SI4825 Band setup example -> Si4827/44 Band setup example
