File: extras/KiCad/SI4844_ATMEGA328_LCD16x02/SI4844_ATMEGA328_LCD16x02.kicad_sch (KiCad schematic)
At the start: 35 parts, among them J1 AudioJack2_Ground, J10 Arduino pin 8, J11 Arduino pin 9, J12 Arduino pin 10, J13 Arduino pin 11, J2 Arduino pin 2, J3 SI4844 pin 2 (IRQ), J4 Arduino pin 12, J5 SI4844 pin 15 (RST), J6 BAND_UP, J7 BAND_DOWN, J8 VOL_UP, J9 VOL_DOWN, U1 LCD16x02, Y1 Crystal

Commit message: Doc
Connections:
- net +3.3V: now also U1.2 (VDD); no longer U1.1 (VSS)
- net GND: now also U1.1 (VSS)
Changed lines of the file:
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@@
+    (stroke (width 0) (type default))
+  )
+  (wire (pts (xy 86.36 63.5) (xy 86.36 66.04))
+    (stroke (width 0) (type default))
+  )
+  (wire (pts (xy 110.49 54.61) (xy 110.49 58.42))
+    (stroke (width 0) (type default))
+  )
+  (wire (pts (xy 222.25 115.57) (xy 229.87 115.57))
     (stroke (width 0) (type default))
   )
@@
     (stroke (width 0) (type default))
   )
-  (wire (pts (xy 86.36 63.5) (xy 86.36 66.04))
-    (stroke (width 0) (type default))
-  )
-  (wire (pts (xy 110.49 54.61) (xy 110.49 58.42))
-    (stroke (width 0) (type default))
-  )
-  (wire (pts (xy 222.25 115.57) (xy 229.87 115.57))
-    (stroke (width 0) (type default))
-  )
   (wire (pts (xy 55.88 68.58) (xy 45.72 68.58))
     (stroke (width 0) (type default))
@@
   )
   (wire (pts (xy 165.1 100.33) (xy 201.93 100.33))
+    (stroke (width 0) (type default))
+  )
+  (wire (pts (xy 212.09 128.27) (xy 212.09 135.89))
     (stroke (width 0) (type default))
   )
@@
     )
   )
+  (symbol (lib_id "power:GND") (at 212.09 85.09 180) (unit 1)
+    (in_bom yes) (on_board yes) (dnp no) (fields_autoplaced)
+    (property "Reference" "#PWR023" (at 212.09 78.74 0)
+      (effects (font (size 1.27 1.27)) hide)
+    )
+    (property "Value" "GND" (at 212.09 80.01 0)
+      (effects (font (size 1.27 1.27)))
+    )
+    (property "Footprint" "" (at 212.09 85.09 0)
+      (effects (font (size 1.27 1.27)) hide)
+    )
+    (property "Datasheet" "" (at 212.09 85.09 0)
+      (effects (font (size 1.27 1.27)) hide)
+    )
+    (pin "1")
+    (instances
+      (project "SI4844_ATMEGA328_LCD16x02"
+        (path "/a0d8c9a3-7eb8-440c-942e-981585e19cdf"
+          (reference "#PWR023") (unit 1)
+        )
+      )
+    )
+  )
   (symbol (lib_id "Connector:Conn_01x01_Pin") (at 172.72 87.63 180) (unit 1)
     (in_bom yes) (on_board yes) (dnp no)
@@
     )
   )
-  (symbol (lib_id "power:+3.3V") (at 212.09 85.09 0) (unit 1)
-    (in_bom yes) (on_board yes) (dnp no) (fields_autoplaced)
-    (property "Reference" "#PWR015" (at 212.09 88.9 0)
-      (effects (font (size 1.27 1.27)) hide)
-    )
-    (property "Value" "+3.3V" (at 212.09 80.01 0)
-      (effects (font (size 1.27 1.27)))
-    )
-    (property "Footprint" "" (at 212.09 85.09 0)
-      (effects (font (size 1.27 1.27)) hide)
-    )
-    (property "Datasheet" "" (at 212.09 85.09 0)
-      (effects (font (size 1.27 1.27)) hide)
-    )
+  (symbol (lib_id "power:+3.3V") (at 212.09 135.89 180) (unit 1)
+    (in_bom yes) (on_board yes) (dnp no) (fields_autoplaced)
+    (property "Reference" "#PWR015" (at 212.09 132.08 0)
+      (effects (font (size 1.27 1.27)) hide)
+    )
+    (property "Value" "+3.3V" (at 214.63 137.16 0)
+      (effects (font (size 1.27 1.27)) (justify right))
+    )
+    (property "Footprint" "" (at 212.09 135.89 0)
+      (effects (font (size 1.27 1.27)) hide)
+    )
+    (property "Datasheet" "" (at 212.09 135.89 0)
+      (effects (font (size 1.27 1.27)) hide)
+    )
